File: hardware/Penguino-STM32WL-M.sch (KiCad schematic (older format))
At the start: 67 parts, among them J1 JST_PH, J2 USB_C_Receptacle_USB2.0, J3 Conn_ARM_JTAG_SWD_10, J4 U.FL-R-SMT-1, J5 SMA-Edge-Mount, Q1 SI2323DS, SW1 RESET, SW2 BOOT0, U1 MCP73831, U2 RT9078-33GJ5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

Commit message: lib: Add iBOM file
Parts:
- C1, C2: MPN 0603B103K500NT -> CC0402KRX7R9BB103
- C10, C13: MPN CL05B104KO5NNNC -> GRM155R61A104KA01D
- C12, C14, C4, C7, C8, C9: MPN CC0603KRX7R9BB104 -> GRM155R61A104KA01D
- C3, C5, C6: MPN CL10A106KP8NNNC -> CC0603KRX5R6BB106
- D1: MPN E6C0603SEAC1UDA -> 19-217-Y5C-AM1N1VY-3T
- D5: MPN ESD0504F -> NUP2202
- J3: MPN (none) -> 20021121-00010C4LF
- J4: MPN U.FL-R-SMT-1(80) -> U.FL-R-SMT-1(80)
- Q1: MPN IRLML6402TRPBF -> SI2323DS
- R1: MPN 0402WGF4701TCE -> RC0402JR-074K7L
- R13, R14, R2: MPN 0402WGF1004TCE -> RC0402JR-071ML
- R4: MPN 0402WGF1003TCE -> RC0402JR-07100KL
- R5, R6, R7: MPN 0402WGF1201TCE -> RC0402JR-071K5L
- U3: MPN MAX809STRG -> TPS3839K33D
- U5: MPN BEMWLE2001 -> MAMWLExx
Changed lines of the file:
@@
 F 3 "~" H 1125 4225 50  0001 C CNN
 F 4 "-" H -350 175 50  0001 C CNN "Mfg"
-F 5 "0402WGF1004TCE" H 1125 4225 50  0001 C CNN "MPN"
+F 5 "RC0402JR-071ML" H 1125 4225 50  0001 C CNN "MPN"
 F 6 "C26083" H 1125 4225 50  0001 C CNN "LCSC_Part#"
 	1    1125 4225
@@
 F 2 "Capacitor_SMD:C_0402_1005Metric" H 813 4050 50  0001 C CNN
 F 3 "~" H 775 4200 50  0001 C CNN
-F 4 "0603B103K500NT" H -400 150 50  0001 C CNN "MPN"
+F 4 "CC0402KRX7R9BB103" H -400 150 50  0001 C CNN "MPN"
 F 5 "C57112" H 775 4200 50  0001 C CNN "LCSC_Part#"
 	1    775  4200
@@
 F 2 "Capacitor_SMD:C_0402_1005Metric" H 2513 2475 50  0001 C CNN
 F 3 "~" H 2475 2625 50  0001 C CNN
-F 4 "0603B103K500NT" H 125 -225 50  0001 C CNN "MPN"
+F 4 "CC0402KRX7R9BB103" H 125 -225 50  0001 C CNN "MPN"
 F 5 "C57112" H 2475 2625 50  0001 C CNN "LCSC_Part#"
 	1    2475 2625
@@
 F 2 "Capacitor_SMD:C_0402_1005Metric" H 3013 2475 50  0001 C CNN
 F 3 "~" H 2975 2625 50  0001 C CNN
-F 4 "CC0603KRX7R9BB104" H 125 -225 50  0001 C CNN "MPN"
+F 4 "GRM155R61A104KA01D" H 125 -225 50  0001 C CNN "MPN"
 F 5 "C14663" H 2975 2625 50  0001 C CNN "LCSC_Part#"
 	1    2975 2625
@@
 F 3 "~" H 1875 1500 50  0001 C CNN
 F 4 "-" H -1400 100 50  0001 C CNN "Mfg"
-F 5 "E6C0603SEAC1UDA" H 1875 1500 50  0001 C CNN "MPN"
+F 5 "19-217-Y5C-AM1N1VY-3T" H 1875 1500 50  0001 C CNN "MPN"
 F 6 "C375450" H 1875 1500 50  0001 C CNN "LCSC_Part#"
 	1    1875 1500
@@
 F 2 "Capacitor_SMD:C_0402_1005Metric" H 5988 5825 50  0001 C CNN
 F 3 "~" H 5950 5975 50  0001 C CNN
-F 4 "CL05B104KO5NNNC" H 125 0   50  0001 C CNN "MPN"
+F 4 "GRM155R61A104KA01D" H 125 0   50  0001 C CNN "MPN"
 F 5 "C1525" H 5950 5975 50  0001 C CNN "LCSC_Part#"
 	1    5950 5975
@@
 F 2 "Package_TO_SOT_SMD:SOT-23" H 5600 1500 50  0001 C CNN
 F 3 "" H 5600 1500 50  0001 C CNN
-F 4 "MAX809STRG" H 1575 25  50  0001 C CNN "MPN"
+F 4 "TPS3839K33D" H 1575 25  50  0001 C CNN "MPN"
 F 5 "C9965" H 5600 1500 50  0001 C CNN "LCSC_Part#"
 	1    5600 1500
@@
 F 2 "Connector_PinHeader_1.27mm:PinHeader_2x05_P1.27mm_Vertical_SMD" H 2450 5475 50  0001 C CNN
 F 3 "http://infocenter.arm.com/help/topic/com.arm.doc.ddi0314h/DDI0314H_coresight_components_trm.pdf" V 2100 4225 50  0001 C CNN
-F 4 "~" H 2450 5475 50  0001 C CNN "MPN"
+F 4 "20021121-00010C4LF" H 2450 5475 50  0001 C CNN "MPN"
 F 5 "~" H 2450 5475 50  0001 C CNN "LCSC_Part#"
 	1    2450 5475
@@
 F 3 "~" H 2450 1250 50  0001 C CNN
 F 4 "-" H -2175 -400 50  0001 C CNN "Mfg"
-F 5 "CL10A106KP8NNNC" H 2450 1250 50  0001 C CNN "MPN"
+F 5 "CC0603KRX5R6BB106" H 2450 1250 50  0001 C CNN "MPN"
 F 6 "C19702" H 2450 1250 50  0001 C CNN "LCSC_Part#"
 	1    2450 1250
@@
 F 2 "Package_TO_SOT_SMD:SOT-23" H 3400 1200 50  0001 C CNN
 F 3 "~" H 3200 1100 50  0001 C CNN
-F 4 "IRLML6402TRPBF" H 3200 1100 50  0001 C CNN "MPN"
+F 4 "SI2323DS" H 3200 1100 50  0001 C CNN "MPN"
 F 5 "C2593" H 3200 1100 50  0001 C CNN "LCSC_Part#"
 	1    3200 1100
@@
 F 3 "~" H 3300 1550 50  0001 C CNN
 F 4 "-" H -1325 -100 50  0001 C CNN "Mfg"
-F 5 "CL10A106KP8NNNC" H 3300 1550 50  0001 C CNN "MPN"
+F 5 "CC0603KRX5R6BB106" H 3300 1550 50  0001 C CNN "MPN"
 F 6 "C19702" H 3300 1550 50  0001 C CNN "LCSC_Part#"
 	1    3300 1550
@@
 F 2 "Resistor_SMD:R_0402_1005Metric" V 640 1665 50  0001 C CNN
 F 3 "~" H 600 1675 50  0001 C CNN
-F 4 "0402WGF4701TCE" H 600 1675 50  0001 C CNN "MPN"
+F 4 "RC0402JR-074K7L" H 600 1675 50  0001 C CNN "MPN"
 F 5 "C25900" H 600 1675 50  0001 C CNN "LCSC_Part#"
 	1    600  1675
@@
 F 2 "Resistor_SMD:R_0402_1005Metric" V 2890 1565 50  0001 C CNN
 F 3 "~" H 2850 1575 50  0001 C CNN
-F 4 "0402WGF1003TCE" H 2850 1575 50  0001 C CNN "MPN"
+F 4 "RC0402JR-07100KL" H 2850 1575 50  0001 C CNN "MPN"
 F 5 "C25741" H 2850 1575 50  0001 C CNN "LCSC_Part#"
 	1    2850 1575
@@
 F 2 "Resistor_SMD:R_0402_1005Metric" V 6290 5565 50  0001 C CNN
 F 3 "~" H 6250 5575 50  0001 C CNN
-F 4 "0402WGF1004TCE" H 6250 5575 50  0001 C CNN "MPN"
+F 4 "RC0402JR-071ML" H 6250 5575 50  0001 C CNN "MPN"
 F 5 "C26083" H 6250 5575 50  0001 C CNN "LCSC_Part#"
 	1    6250 5575
@@
 F 2 "Resistor_SMD:R_0402_1005Metric" V 6290 5965 50  0001 C CNN
 F 3 "~" H 6250 5975 50  0001 C CNN
-F 4 "0402WGF1004TCE" H 6250 5975 50  0001 C CNN "MPN"
+F 4 "RC0402JR-071ML" H 6250 5975 50  0001 C CNN "MPN"
 	1    6250 5975
 	1    0    0    -1
@@
 F 2 "Resistor_SMD:R_0402_1005Metric" V 4290 3590 50  0001 C CNN
 F 3 "~" H 4250 3600 50  0001 C CNN
-F 4 "0402WGF1201TCE" H 4250 3600 50  0001 C CNN "MPN"
+F 4 "RC0402JR-071K5L" H 4250 3600 50  0001 C CNN "MPN"
 F 5 "C25862" H 4250 3600 50  0001 C CNN "LCSC_Part#"
 	1    4250 3600
@@
 F 2 "Resistor_SMD:R_0402_1005Metric" V 4490 3590 50  0001 C CNN
 F 3 "~" H 4450 3600 50  0001 C CNN
-F 4 "0402WGF1201TCE" H 4450 3600 50  0001 C CNN "MPN"
+F 4 "RC0402JR-071K5L" H 4450 3600 50  0001 C CNN "MPN"
 F 5 "C25862" H 4450 3600 50  0001 C CNN "LCSC_Part#"
 	1    4450 3600
@@
 F 2 "Resistor_SMD:R_0402_1005Metric" V 4690 3590 50  0001 C CNN
 F 3 "~" H 4650 3600 50  0001 C CNN
-F 4 "0402WGF1201TCE" H 4650 3600 50  0001 C CNN "MPN"
+F 4 "RC0402JR-071K5L" H 4650 3600 50  0001 C CNN "MPN"
 F 5 "C25862" H 4650 3600 50  0001 C CNN "LCSC_Part#"
 	1    4650 3600
@@
 F 2 "stm32wl-lib-v1:stm32wl-mamwlexx-module-footprint_w_s_paste" H 8125 1775 50  0001 C CNN
 F 3 "" H 8125 1775 50  0001 C CNN
-F 4 "BEMWLE2001" H 8125 1775 50  0001 C CNN "MPN"
+F 4 "MAMWLExx" H 8125 1775 50  0001 C CNN "MPN"
 	1    8125 1775
 	1    0    0    -1
@@
 F 2 "Connector_Coaxial:U.FL_Hirose_U.FL-R-SMT-1_Vertical" H 8775 675 50  0001 C CNN
 F 3 " ~" H 8775 675 50  0001 C CNN
-F 4 " U.FL-R-SMT-1(80)" H 8775 675 50  0001 C CNN "MPN"
+F 4 "U.FL-R-SMT-1(80)" H 8775 675 50  0001 C CNN "MPN"
 F 5 "~" H 8775 675 50  0001 C CNN "LCSC_Part#"
 	1    8775 675
@@
 F 2 "Capacitor_SMD:C_0402_1005Metric" H 5063 1500 50  0001 C CNN
 F 3 "~" H 5025 1650 50  0001 C CNN
-F 4 "CC0603KRX7R9BB104" H 2175 -1200 50  0001 C CNN "MPN"
+F 4 "GRM155R61A104KA01D" H 2175 -1200 50  0001 C CNN "MPN"
 F 5 "C14663" H 5025 1650 50  0001 C CNN "LCSC_Part#"
 	1    5025 1650
@@
 F 3 "~" H 4800 1650 50  0001 C CNN
 F 4 "-" H -1350 0   50  0001 C CNN "Mfg"
-F 5 "CL10A106KP8NNNC" H 4800 1650 50  0001 C CNN "MPN"
+F 5 "CC0603KRX5R6BB106" H 4800 1650 50  0001 C CNN "MPN"
 F 6 "C19702" H 4800 1650 50  0001 C CNN "LCSC_Part#"
 	1    4800 1650
@@
 F 2 "Package_TO_SOT_SMD:SOT-363_SC-70-6" H 2855 3775 50  0001 C CNN
 F 3 "" H 2855 3775 50  0001 C CNN
-F 4 "ESD0504F" H 2775 3700 50  0001 C CNN "MPN"
+F 4 "NUP2202" H 2775 3700 50  0001 C CNN "MPN"
 F 5 "C502602" H 2775 3700 50  0001 C CNN "LCSC_Part#"
 	1    2775 3700
@@
 F 2 "Capacitor_SMD:C_0402_1005Metric" H 7963 4525 50  0001 C CNN
 F 3 "~" H 7925 4675 50  0001 C CNN
-F 4 "CL05B104KO5NNNC" H 5075 1825 50  0001 C CNN "MPN"
+F 4 "GRM155R61A104KA01D" H 5075 1825 50  0001 C CNN "MPN"
 F 5 "C1525" H 7925 4675 50  0001 C CNN "LCSC_Part#"
 	1    7925 4675
@@
 F 2 "Capacitor_SMD:C_0402_1005Metric" H 6863 3675 50  0001 C CNN
 F 3 "~" H 6825 3825 50  0001 C CNN
-F 4 "CC0603KRX7R9BB104" H 3975 975 50  0001 C CNN "MPN"
+F 4 "GRM155R61A104KA01D" H 3975 975 50  0001 C CNN "MPN"
 F 5 "C14663" H 6825 3825 50  0001 C CNN "LCSC_Part#"
 	1    6825 3825
@@
 F 2 "Capacitor_SMD:C_0402_1005Metric" H 7138 3675 50  0001 C CNN
 F 3 "~" H 7100 3825 50  0001 C CNN
-F 4 "CC0603KRX7R9BB104" H 4250 975 50  0001 C CNN "MPN"
+F 4 "GRM155R61A104KA01D" H 4250 975 50  0001 C CNN "MPN"
 F 5 "C14663" H 7100 3825 50  0001 C CNN "LCSC_Part#"
 	1    7100 3825
@@
 F 2 "Capacitor_SMD:C_0402_1005Metric" H 7463 3675 50  0001 C CNN
 F 3 "~" H 7425 3825 50  0001 C CNN
-F 4 "CC0603KRX7R9BB104" H 4575 975 50  0001 C CNN "MPN"
+F 4 "GRM155R61A104KA01D" H 4575 975 50  0001 C CNN "MPN"
 F 5 "C14663" H 7425 3825 50  0001 C CNN "LCSC_Part#"
 	1    7425 3825
@@
 F 2 "Capacitor_SMD:C_0402_1005Metric" H 5988 3700 50  0001 C CNN
 F 3 "~" H 5950 3850 50  0001 C CNN
-F 4 "CC0603KRX7R9BB104" H 3100 1000 50  0001 C CNN "MPN"
+F 4 "GRM155R61A104KA01D" H 3100 1000 50  0001 C CNN "MPN"
 F 5 "C14663" H 5950 3850 50  0001 C CNN "LCSC_Part#"
 	1    5950 3850
