File: hardware/Penguino-STM32WL-M.kicad_pcb (KiCad board)
At the start: 4 copper layers, 22.9 x 50.8 mm, 68 parts, among them J1 JST_PH, J2 USB_C_Receptacle_USB2.0, J3 Conn_ARM_JTAG_SWD_10, J4 U.FL-R-SMT-1, J5 SMA-Edge-Mount, Q1 SI2323DS, SW1 RESET, SW2 BOOT0, U1 MCP73831, U2 RT9078-33GJ5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

Commit message: hw, fw: Examples added, KiCAD version upgraded
Routing:
- added copper zone on In2.Cu, net +3V3
- added copper zone on In1.Cu, net GND
- removed copper zone on In2.PWR, net +3V3
- removed copper zone on In1.GND, net GND
Other:
- net class Default removed
